File: hardware/data-capture.sch (KiCad schematic (older format))
At the start: 49 parts, among them J3 DM3AT-SF-PEJM5, J4 Conn_01x02, Q1 Q_PMOS_GSD, SW1 SW_Push, U1 MCP73831-2-OT, U2 TLV70218_SOT23-5, U3 AP2112K-3.3, U4 MDBT50Q-1M, U5 PCA9306, U6 ICM-20948, U7 BMP280, Y1 32.768

Commit message: update schematic for ESYNC for IMU
Parts:
- J1: renamed from J?; symbol Connector_Specialized:USB_B_Mini -> data-capture-rescue:USB_B_Mini-Connector_Specialized
- U2: symbol Regulator_Linear:TLV70218_SOT23-5 -> data-capture-rescue:TLV70218_SOT23-5-Regulator_Linear
- gave numbers to parts that had none: 1
Connections:
- net GND: no longer U6.11 (FSYNC)
- net IMU_FSYC: now reaches U4.4 (P1.11)
- net IMU_FSYC: now also U6.11 (FSYNC)
Changed lines of the file:
@@
 EESchema Schematic File Version 4
-EELAYER 29 0
+EELAYER 30 0
 EELAYER END
 $Descr A4 11693 8268
@@
 	4350 1050 4450 1050
 $Comp
-L Regulator_Linear:TLV70218_SOT23-5 U2
+L data-capture-rescue:TLV70218_SOT23-5-Regulator_Linear U2
 U 1 1 5C9FA53F
 P 1900 3800
@@
 F 3 "" H 9000 2000 50  0001 C CNN
 	1    9000 2000
-	0    1    1    0
-$EndComp
-$Comp
-L power:GND #PWR0145
-U 1 1 5CA160C4
-P 9000 1600
-F 0 "#PWR0145" H 9000 1350 50  0001 C CNN
-F 1 "GND" V 9005 1472 50  0000 R CNN
-F 2 "" H 9000 1600 50  0001 C CNN
-F 3 "" H 9000 1600 50  0001 C CNN
-	1    9000 1600
 	0    1    1    0
 $EndComp
@@
 NEO_LED
 $Comp
-L bed-sensor-rescue:Conn_ARM_JTAG_SWD_10-Connector_Specialized-bed-sensor-rescue-bed-sensor-rescue-bed-sensor-rescue-bed-sensor-rescue-bed-sensor-rescue-bed-sensor-rescue-bed-sensor-rescue-bed-sensor-rescue-bed-sensor-rescue J?
+L bed-sensor-rescue:Conn_ARM_JTAG_SWD_10-Connector_Specialized-bed-sensor-rescue-bed-sensor-rescue-bed-sensor-rescue-bed-sensor-rescue-bed-sensor-rescue-bed-sensor-rescue-bed-sensor-rescue-bed-sensor-rescue-bed-sensor-rescue J2
 U 1 1 5D0BD668
 P 2950 6150
-F 0 "J?" H 2507 6196 50  0000 R CNN
+F 0 "J2" H 2507 6196 50  0000 R CNN
 F 1 "Conn_ARM_JTAG_SWD_10-Connector_Specialized-bed-sensor-rescue-bed-sensor-rescue-bed-sensor-rescue-bed-sensor-rescue-bed-sensor-rescue-bed-sensor-rescue-bed-sensor-rescue-bed-sensor-rescue-bed-sensor-rescue" H 2507 6105 50  0000 R CNN
 F 2 "Connector_PinHeader_1.27mm:PinHeader_2x05_P1.27mm_Vertical_SMD" H 3000 5600 50  0001 L TNN
@@
 Connection ~ 2850 6750
 $Comp
-L Connector_Specialized:USB_B_Mini J?
+L data-capture-rescue:USB_B_Mini-Connector_Specialized J1
 U 1 1 5D0BFDB4
 P 1100 5800
-F 0 "J?" H 1157 6267 50  0000 C CNN
+F 0 "J1" H 1157 6267 50  0000 C CNN
 F 1 "USB_B_Mini" H 1157 6176 50  0000 C CNN
 F 2 "" H 1250 5750 50  0001 C CNN
@@
 $EndComp
 Connection ~ 1000 6200
+Text GLabel 3550 3400 0    50   Input ~ 0
+IMU_FSYC
+Text GLabel 9000 1600 0    50   Input ~ 0
+IMU_FSYC
 $EndSCHEMATC
